Commit message: 드론 자율비행 — 층별 지도 + 전역 층 선택 + 지역 고도 회피
Nav2 는 2D 라 고도를 계획하지 않는다. 그 한 축만 바깥에서 담당해 "장애물을
넘어간다" 를 얻는다. Nav2 자체는 고치지 않고 인자 두 개만 바꿔 끼운다.

- drone_layer_mapper: 라이다+하향 뎁스 -> 층(1/2/3 m)별 점유 격자.
  slam_toolbox 를 뺐다 — odom 이 이미 월드 절대좌표라 점유 격자 누적기로만
  쓰이고 있었다. map(층 합집합, 병합기용) / map_active(현재 층, Nav2) /
  map_layer_k(후보 층) 로 나눈 이유는 소비자가 서로 다른 것을 봐야 해서다.
- altitude_selector: 목표까지 회랑을 층마다 검사해 순항 고도 결정.
  하드 실패로 두면 아무 층도 안 뚫려서(108개 방향 중 0개) 비율 기준으로 바꿨다.
- local_altitude_avoider: 룩어헤드 3 m 감시 -> linear.z 합성, cmd_vel 단독 발행.
  복귀 판정은 "지금 비었나" 가 아니라 "순항 고도로 내려가도 되나" 다 —
  전자로 두면 리밋 사이클에 빠진다. 하향 센서를 하강 판단에 연결해 장애물
  위에 착지하는 것도 막는다.
- NAV_MODE 환경 변수로 2d / 2.5d_local / 2.5d 를 고른다 (compose 가 넣어 준다)
- 드론 PROTO 를 래퍼(Mavic2ProMediumSensorized)로 교체 — 라이다가 그 안에 있다

실측: 목표 5개 중 4개 도달(오차 0.07~0.22 m), 방향전환 0회.
자세한 것은 DRONE_NAV.md.

Co-Authored-By: Claude Opus 5 <noreply@anthropic.com>

File: src/webots_python/urdf/Mavic2ProMedium.urdf.xacro (robot description, xacro)
@@ -51,8 +51,45 @@
     <origin xyz="0 0 0" rpy="0 0 0"/>
   </joint>
+  <!-- 라이다: 동체 위 0.12 m. Mavic2ProMediumSensorized.proto 의 bodySlot 위치와
+       **같아야 한다** — 여기가 어긋나면 스캔이 실제와 다른 곳에서 나온 것처럼 변환되어
+       SLAM 이 조용히 틀린 맵을 그린다. 그 높이를 왜 0.12 로 골랐는지는 PROTO 주석 참고. -->
+  <link name="Velodyne_VLP_16">
+    <visual>
+      <geometry>
+        <cylinder radius="0.052" length="0.0727"/>
+      </geometry>
+    </visual>
+  </link>
+  <joint name="base_link_Velodyne_VLP_16_joint" type="fixed">
+    <parent link="base_link"/>
+    <child link="Velodyne_VLP_16"/>
+    <origin xyz="0 0 0.12" rpy="0 0 0"/>
+  </joint>
+  <!-- 하향 뎁스센서: 동체 아래 0.12 m, 정면(+x)이 아래(-z)를 보도록 y축 +90° 회전.
+       PROTO 의 배치와 **같아야 한다** (라이다와 같은 이유). -->
+  <link name="down_depth"/>
+  <joint name="base_link_down_depth_joint" type="fixed">
+    <parent link="base_link"/>
+    <child link="down_depth"/>
+    <origin xyz="-0.12 0 -0.12" rpy="0 1.5708 0"/>
+  </joint>
   <webots>
     <plugin type="simulator.drone_driver.main">
       <namespace>$(arg namespace)</namespace>
     </plugin>
+    <!-- 라이다는 Mavic2ProMediumSensorized.proto 에만 있다. 순정 Mavic2ProMedium 을
+         손으로 놓고 이 URDF 를 쓰면 드라이버가 "device not found" 경고만 내고 넘어간다
+         (치명적이지 않지만 그 드론은 SLAM 을 못 돌린다). -->
+    <device reference="Velodyne_VLP_16" type="Lidar">
+      <ros><frameName>$(arg namespace)/Velodyne_VLP_16</frameName></ros>
+    </device>
+    <!-- 하향 뎁스센서. 층 선택기가 /{ns}/down_depth/point_cloud 로 발밑을 본다. -->
+    <device reference="down_depth" type="RangeFinder">
+      <ros>
+        <topicName>/$(arg namespace)/down_depth</topicName>
+        <frameName>$(arg namespace)/down_depth</frameName>
+        <enabled>true</enabled>
+      </ros>
+    </device>
     <device reference="camera" type="Camera">
       <ros>
